Commit message: Adding Lidar to the URDF and resolving conflicts with collisions for MoveIt!

File: ros-stacks/motoman/motoman_hc10_support/urdf/hc10dt_macro.xacro (robot description, xacro)
@@ -2,4 +2,8 @@
 <robot xmlns:xacro="http://ros.org/wiki/xacro">
   <xacro:macro name="motoman_hc10dt" params="prefix">
+  <!-- Adhiti Additions -->
+  <xacro:arg name="gpu" default="false"/>
+  <xacro:property name="gpu" value="$(arg gpu)" />
+  <!-- end -->
     <!-- Properties -->
     <material name="yaskawa_blue">
@@ -131,4 +135,5 @@
     <link name="${prefix}tool0"/>
     <!-- end of link list -->
+  <!-- end -->
     <!-- joint list -->
     <joint name="${prefix}joint_1_s" type="revolute">
@@ -187,4 +192,10 @@
       <child link="${prefix}base"/>
     </joint>
+  <!-- Adding the lidar marcos -->
+    <xacro:include filename="$(find velodyne_description)/urdf/VLP-16.urdf.xacro"/>
+    <VLP-16 parent="${prefix}tool0" name="velodyne" topic="/velodyne_points" hz="10" samples="440" gpu="${gpu}">
+      <origin xyz="0 0 0" rpy="0 0 0" />
+    </VLP-16>
+  <!-- end -->
   </xacro:macro>
 </robot>
